Commit message: Adding collision model

File: urdf/ewellix_lift_500mm.urdf.xacro (robot description, xacro)
@@ -32,7 +32,7 @@
       </visual>
       <collision>
-        <origin xyz="0.0 0 0.0" rpy="0 0 ${M_PI/2}"/>
+        <origin xyz="0.000 -0.035 0.188" rpy="0 0 ${M_PI/2}"/>
         <geometry>
-          <mesh filename="package://ewellix_tlt/meshes/ewellix_lift_base_500mm.stl"  scale="0.001 0.001 0.001"/>
+          <box size="0.163 0.234 0.376"/>
         </geometry>
       </collision>
@@ -66,11 +66,13 @@
       </visual>
       <collision>
-        <origin xyz="0.0 0 0.0" rpy="0 0 -${M_PI/2}"/>
+        <origin xyz="0.0 0 -0.3515" rpy="0 0 -${M_PI/2}"/>
         <geometry>
           <xacro:if value="${cut_model}">
-            <mesh filename="package://ewellix_tlt/meshes/ewellix_lift_top_500mm.stl" scale="0.001 0.001 0.001"/>
+            <!-- <mesh filename="package://ewellix_tlt/meshes/ewellix_lift_top_500mm.stl" scale="0.001 0.001 0.001"/> -->
+            <box size="0.146 0.146 0.703"/>
           </xacro:if>
           <xacro:unless value="${cut_model}">
-            <mesh filename="package://ewellix_tlt/meshes/ewellix_lift_top_500mm.stl" scale="0.001 0.001 0.001"/>
+            <!-- <mesh filename="package://ewellix_tlt/meshes/ewellix_lift_top_500mm.stl" scale="0.001 0.001 0.001"/> -->
+            <box size="0.146 0.146 0.703"/>
           </xacro:unless>
         </geometry>

Commit message: Tightened collision model

File: urdf/ewellix_lift_500mm.urdf.xacro (robot description, xacro)
@@ -32,7 +32,7 @@
       </visual>
       <collision>
-        <origin xyz="0.000 -0.035 0.188" rpy="0 0 ${M_PI/2}"/>
+        <origin xyz="0.000 0.000 0.188" rpy="0 0 ${M_PI/2}"/>
         <geometry>
-          <box size="0.163 0.234 0.376"/>
+          <box size="0.163 0.163 0.376"/>
         </geometry>
       </collision>
